Commit message: V1.1—优化1

File: assets/robots/ur5_allegro/ur5_allegro.urdf (robot description, URDF)
Before this commit: robot ur5, 35 links, 34 joints
Links:
- removed link Link_1
- removed link platform_base_link
- removed link world
Joints:
- removed joint Link_1
- removed joint platform2ur5_joint
- removed joint worldur5_to_base
